Commit message: modify my_robot_simulation

File: src/my_robot_description/urdf/robotiq.ros2_control.xacro (robot description, xacro)
@@ -3,5 +3,5 @@
     <xacro:macro name="robotiq_gripper_ros2_control" params="
         name
-        prefix
+        tf_prefix
         sim_gazebo:=false
         sim_ignition:=false
@@ -51,5 +51,5 @@
             <!-- Joint interfaces -->
             <!-- With Ignition or Hardware, they handle mimic joints, so we only need this command interface activated -->
-            <joint name="${prefix}robotiq_85_left_knuckle_joint">
+            <joint name="${tf_prefix}robotiq_85_left_knuckle_joint">
                 <command_interface name="position" />
                 <state_interface name="position">
@@ -61,6 +61,6 @@
             <!-- When simulating we need to include the rest of the gripper joints -->
             <xacro:if value="${sim_gazebo or use_fake_hardware or sim_isaac or sim_ignition}">
-                <joint name="${prefix}robotiq_85_right_knuckle_joint">
-                    <param name="mimic">${prefix}robotiq_85_left_knuckle_joint</param>
+                <joint name="${tf_prefix}robotiq_85_right_knuckle_joint">
+                    <param name="mimic">${tf_prefix}robotiq_85_left_knuckle_joint</param>
                     <param name="multiplier">-1</param>
                     <xacro:unless value="${sim_ignition}">
@@ -70,6 +70,6 @@
                     </xacro:unless>
                 </joint>
-                <joint name="${prefix}robotiq_85_left_inner_knuckle_joint">
-                    <param name="mimic">${prefix}robotiq_85_left_knuckle_joint</param>
+                <joint name="${tf_prefix}robotiq_85_left_inner_knuckle_joint">
+                    <param name="mimic">${tf_prefix}robotiq_85_left_knuckle_joint</param>
                     <param name="multiplier">1</param>
                     <xacro:unless value="${sim_ignition}">
@@ -79,6 +79,6 @@
                     </xacro:unless>
                 </joint>
-                <joint name="${prefix}robotiq_85_right_inner_knuckle_joint">
-                    <param name="mimic">${prefix}robotiq_85_left_knuckle_joint</param>
+                <joint name="${tf_prefix}robotiq_85_right_inner_knuckle_joint">
+                    <param name="mimic">${tf_prefix}robotiq_85_left_knuckle_joint</param>
                     <param name="multiplier">-1</param>
                     <xacro:unless value="${sim_ignition}">
@@ -88,6 +88,6 @@
                     </xacro:unless>
                 </joint>
-                <joint name="${prefix}robotiq_85_left_finger_tip_joint">
-                    <param name="mimic">${prefix}robotiq_85_left_knuckle_joint</param>
+                <joint name="${tf_prefix}robotiq_85_left_finger_tip_joint">
+                    <param name="mimic">${tf_prefix}robotiq_85_left_knuckle_joint</param>
                     <param name="multiplier">-1</param>
                     <xacro:unless value="${sim_ignition}">
@@ -97,6 +97,6 @@
                     </xacro:unless>
                 </joint>
-                <joint name="${prefix}robotiq_85_right_finger_tip_joint">
-                    <param name="mimic">${prefix}robotiq_85_left_knuckle_joint</param>
+                <joint name="${tf_prefix}robotiq_85_right_finger_tip_joint">
+                    <param name="mimic">${tf_prefix}robotiq_85_left_knuckle_joint</param>
                     <param name="multiplier">1</param>
                     <xacro:unless value="${sim_ignition}">

File: src/my_robot_description/urdf/robotiq_macro.urdf.xacro (robot description, xacro)
@@ -3,5 +3,5 @@
     <xacro:macro name="robotiq_gripper" params="
         name
-        prefix
+        tf_prefix
         parent
         *origin
@@ -25,5 +25,5 @@
         <xacro:if value="${include_ros2_control}">
             <xacro:robotiq_gripper_ros2_control
-                name="${name}" prefix="${prefix}"
+                name="${name}" tf_prefix="${tf_prefix}"
                 sim_gazebo="${sim_gazebo}"
                 sim_ignition="${sim_ignition}"
@@ -40,5 +40,5 @@
                 gripper_closed_position="${gripper_closed_position}"/>
         </xacro:if>
-        <link name="${prefix}robotiq_85_base_link">
+        <link name="${tf_prefix}robotiq_85_base_link">
             <visual>
                 <geometry>
@@ -57,5 +57,5 @@
             </inertial>
         </link>
-        <link name="${prefix}robotiq_85_left_knuckle_link">
+        <link name="${tf_prefix}robotiq_85_left_knuckle_link">
             <visual>
                 <geometry>
@@ -74,5 +74,5 @@
             </inertial>
         </link>
-        <link name="${prefix}robotiq_85_right_knuckle_link">
+        <link name="${tf_prefix}robotiq_85_right_knuckle_link">
             <visual>
                 <geometry>
@@ -91,5 +91,5 @@
             </inertial>
         </link>
-        <link name="${prefix}robotiq_85_left_finger_link">
+        <link name="${tf_prefix}robotiq_85_left_finger_link">
             <visual>
                 <geometry>
@@ -108,5 +108,5 @@
             </inertial>
         </link>
-        <link name="${prefix}robotiq_85_right_finger_link">
+        <link name="${tf_prefix}robotiq_85_right_finger_link">
             <visual>
                 <geometry>
@@ -125,5 +125,5 @@
             </inertial>
         </link>
-        <link name="${prefix}robotiq_85_left_inner_knuckle_link">
+        <link name="${tf_prefix}robotiq_85_left_inner_knuckle_link">
             <visual>
                 <geometry>
@@ -142,5 +142,5 @@
             </inertial>
         </link>
-        <link name="${prefix}robotiq_85_right_inner_knuckle_link">
+        <link name="${tf_prefix}robotiq_85_right_inner_knuckle_link">
             <visual>
                 <geometry>
@@ -159,5 +159,5 @@
             </inertial>
         </link>
-        <link name="${prefix}robotiq_85_left_finger_tip_link">
+        <link name="${tf_prefix}robotiq_85_left_finger_tip_link">
             <visual>
                 <geometry>
@@ -194,5 +194,5 @@
             </inertial>
         </link>
-        <link name="${prefix}robotiq_85_right_finger_tip_link">
+        <link name="${tf_prefix}robotiq_85_right_finger_tip_link">
             <visual>
                 <geometry>
@@ -229,61 +229,61 @@
             </inertial>
         </link>
-        <joint name="${prefix}robotiq_85_base_joint" type="fixed">
+        <joint name="${tf_prefix}robotiq_85_base_joint" type="fixed">
             <parent link="${parent}" />
-            <child link="${prefix}robotiq_85_base_link" />
+            <child link="${tf_prefix}robotiq_85_base_link" />
             <xacro:insert_block name="origin" />
         </joint>
-        <joint name="${prefix}robotiq_85_left_knuckle_joint" type="revolute">
-            <parent link="${prefix}robotiq_85_base_link" />
-            <child link="${prefix}robotiq_85_left_knuckle_link" />
+        <joint name="${tf_prefix}robotiq_85_left_knuckle_joint" type="revolute">
+            <parent link="${tf_prefix}robotiq_85_base_link" />
+            <child link="${tf_prefix}robotiq_85_left_knuckle_link" />
             <axis xyz="0 -1 0" />
             <origin xyz="0.03060114 0.0 0.05490452" rpy="0 0 0" />
             <limit lower="0.0" upper="0.8" velocity="0.5" effort="50" />
         </joint>
-        <joint name="${prefix}robotiq_85_right_knuckle_joint" type="revolute">
-            <parent link="${prefix}robotiq_85_base_link" />
-            <child link="${prefix}robotiq_85_right_knuckle_link" />
+        <joint name="${tf_prefix}robotiq_85_right_knuckle_joint" type="revolute">
+            <parent link="${tf_prefix}robotiq_85_base_link" />
+            <child link="${tf_prefix}robotiq_85_right_knuckle_link" />
             <axis xyz="0 -1 0" />
             <origin xyz="-0.03060114 0.0 0.05490452" rpy="0 0 0" />
             <limit lower="-0.8" upper="0.0" velocity="0.5" effort="50" />
-            <mimic joint="${prefix}robotiq_85_left_knuckle_joint" multiplier="-1" />
-        </joint>
-        <joint name="${prefix}robotiq_85_left_finger_joint" type="fixed">
-            <parent link="${prefix}robotiq_85_left_knuckle_link" />
-            <child link="${prefix}robotiq_85_left_finger_link" />
+            <mimic joint="${tf_prefix}robotiq_85_left_knuckle_joint" multiplier="-1" />
+        </joint>
+        <joint name="${tf_prefix}robotiq_85_left_finger_joint" type="fixed">
+            <parent link="${tf_prefix}robotiq_85_left_knuckle_link" />
+            <child link="${tf_prefix}robotiq_85_left_finger_link" />
             <origin xyz="0.03152616 0.0 -0.00376347" rpy="0 0 0" />
         </joint>
-        <joint name="${prefix}robotiq_85_right_finger_joint" type="fixed">
-            <parent link="${prefix}robotiq_85_right_knuckle_link" />
-            <child link="${prefix}robotiq_85_right_finger_link" />
+        <joint name="${tf_prefix}robotiq_85_right_finger_joint" type="fixed">
+            <parent link="${tf_prefix}robotiq_85_right_knuckle_link" />
+            <child link="${tf_prefix}robotiq_85_right_finger_link" />
             <origin xyz="-0.03152616 0.0 -0.00376347" rpy="0 0 0" />
         </joint>
-        <joint name="${prefix}robotiq_85_left_inner_knuckle_joint" type="continuous">
-            <parent link="${prefix}robotiq_85_base_link" />
-            <child link="${prefix}robotiq_85_left_inner_knuckle_link" />
+        <joint name="${tf_prefix}robotiq_85_left_inner_knuckle_joint" type="continuous">
+            <parent link="${tf_prefix}robotiq_85_base_link" />
+            <child link="${tf_prefix}robotiq_85_left_inner_knuckle_link" />
             <axis xyz="0 -1 0" />
             <origin xyz="0.0127 0.0 0.06142" rpy="0 0 0" />
-            <mimic joint="${prefix}robotiq_85_left_knuckle_joint" />
-        </joint>
-        <joint name="${prefix}robotiq_85_right_inner_knuckle_joint" type="continuous">
-            <parent link="${prefix}robotiq_85_base_link" />
-            <child link="${prefix}robotiq_85_right_inner_knuckle_link" />
+            <mimic joint="${tf_prefix}robotiq_85_left_knuckle_joint" />
+        </joint>
+        <joint name="${tf_prefix}robotiq_85_right_inner_knuckle_joint" type="continuous">
+            <parent link="${tf_prefix}robotiq_85_base_link" />
+            <child link="${tf_prefix}robotiq_85_right_inner_knuckle_link" />
             <axis xyz="0 -1 0" />
             <origin xyz="-0.0127 0.0 0.06142" rpy="0 0 0" />
-            <mimic joint="${prefix}robotiq_85_left_knuckle_joint" multiplier="-1" />
-        </joint>
-        <joint name="${prefix}robotiq_85_left_finger_tip_joint" type="continuous">
-            <parent link="${prefix}robotiq_85_left_finger_link" />
-            <child link="${prefix}robotiq_85_left_finger_tip_link" />
+            <mimic joint="${tf_prefix}robotiq_85_left_knuckle_joint" multiplier="-1" />
+        </joint>
+        <joint name="${tf_prefix}robotiq_85_left_finger_tip_joint" type="continuous">
+            <parent link="${tf_prefix}robotiq_85_left_finger_link" />
+            <child link="${tf_prefix}robotiq_85_left_finger_tip_link" />
             <axis xyz="0 -1 0" />
             <origin xyz="0.00563134 0.0 0.04718515" rpy="0 0 0" />
-            <mimic joint="${prefix}robotiq_85_left_knuckle_joint" multiplier="-1" />
-        </joint>
-        <joint name="${prefix}robotiq_85_right_finger_tip_joint" type="continuous">
-            <parent link="${prefix}robotiq_85_right_finger_link" />
-            <child link="${prefix}robotiq_85_right_finger_tip_link" />
+            <mimic joint="${tf_prefix}robotiq_85_left_knuckle_joint" multiplier="-1" />
+        </joint>
+        <joint name="${tf_prefix}robotiq_85_right_finger_tip_joint" type="continuous">
+            <parent link="${tf_prefix}robotiq_85_right_finger_link" />
+            <child link="${tf_prefix}robotiq_85_right_finger_tip_link" />
             <axis xyz="0 -1 0" />
             <origin xyz="-0.00563134 0.0 0.04718515" rpy="0 0 0" />
-            <mimic joint="${prefix}robotiq_85_left_knuckle_joint" />
+            <mimic joint="${tf_prefix}robotiq_85_left_knuckle_joint" />
         </joint>
     </xacro:macro>

File: src/my_robot_description/urdf/ur_robotiq_ft.urdf.xacro (robot description, xacro)
@@ -142,6 +142,11 @@
   <xacro:arg name="com_port" default="/dev/ttyUSB0" />
   <!-- Import macros -->
+  <xacro:include filename="$(find my_robot_description)/urdf/robotiq_ft300.urdf.xacro" />
+   <xacro:robotiq_ft300 parent="tool0" tf_prefix="$(arg tf_prefix)">
+    <origin xyz="0 0 0" rpy="0 0 0"/>
+  </xacro:robotiq_ft300>
+  <!-- Import macros -->
   <xacro:include filename="$(find my_robot_description)/urdf/robotiq_macro.urdf.xacro" />
-  <xacro:robotiq_gripper name="RobotiqGripperHardwareInterface" prefix="" parent="tool0" use_fake_hardware="$(arg use_fake_hardware)" com_port="$(arg com_port)" sim_ignition="$(arg sim_ignition)">
+  <xacro:robotiq_gripper name="RobotiqGripperHardwareInterface" tf_prefix=""  parent="robotiq_ft_frame_id" use_fake_hardware="$(arg use_fake_hardware)" com_port="$(arg com_port)" sim_ignition="$(arg sim_ignition)">
     <origin xyz="0 0 0" rpy="0 0 0" />
   </xacro:robotiq_gripper>
